Commit message: added new sensors

File: ros/src/udacity_bot/urdf/udacity_bot.xacro (robot description, xacro)
@@ -1,4 +1,5 @@
 <?xml version='1.0'?>
 <robot name="udacity_bot" xmlns:xacro="http://www.ros.org/wiki/xacro">
+  <xacro:include filename="$(find udacity_bot)/urdf/udacity_bot.gazebo" />
   <link name="robot_footprint"></link>
   <joint name="robot_footprint_joint" type="fixed">
@@ -23,4 +24,5 @@
         <box size=".4 .2 .1"/>
       </geometry>
+       <material name="blue"/>
     </collision>
     <visual name='chassis_visual'>
@@ -35,4 +37,14 @@
         <sphere radius="0.0499"/>
       </geometry>
+      <surface>
+        <friction>
+          <ode>
+            <mu>0</mu>
+            <mu2>0</mu2>
+            <slip1>1.0</slip1>
+            <slip2>1.0</slip2>
+          </ode>
+        </friction>
+      </surface>
     </collision>
     <visual name='back_caster_visual'>
@@ -47,4 +59,14 @@
         <sphere radius="0.0499"/>
       </geometry>
+      <surface>
+        <friction>
+          <ode>
+            <mu>0</mu>
+            <mu2>0</mu2>
+            <slip1>1.0</slip1>
+            <slip2>1.0</slip2>
+          </ode>
+        </friction>
+      </surface>
     </collision>
     <visual name='front_caster_visual'>
@@ -55,3 +77,132 @@
     </visual>
   </link>
+  <!-- Left Wheel -->
+  <link name="left_wheel">
+    <pose>0 0 0 0 1.5707 1.5707</pose>
+    <inertial>
+       <mass value="5.0"/>
+          <origin xyz="0 0 0" rpy="0 1.5707 1.5707"/>
+	     <inertia
+		  ixx="0.1" ixy="0" ixz="0"
+		  iyy="0.1" iyz="0"
+		  izz="0.1"
+	      />
+    </inertial>
+    <collision>
+       <origin xyz="0 0 0" rpy="0 1.5707 1.5707" />
+       <geometry>
+          <cylinder radius="0.1" length="0.05" />
+       </geometry>
+    </collision>
+    <visual>
+       <origin xyz="0 0 0" rpy="0 1.5707 1.5707" />
+       <geometry>
+          <cylinder radius="0.1" length="0.05" />
+       </geometry>
+       <material name="green"/>
+    </visual>
+  </link>
+  <!-- Left Wheel Robot chassis joint -->
+  <joint type="continuous" name="left_wheel_hinge">
+    <origin xyz="0 0.15 0" rpy="0 0 0"/>
+    <child link="left_wheel"/>
+    <parent link="chassis"/>
+    <axis xyz="0 1 0" rpy="0 0 0"/>
+    <limit effort="10000" velocity="1000"/>
+    <joint_properties damping="1.0" friction="1.0"/>
+  </joint>
+  <!-- Right Wheel -->
+  <link name="right_wheel">
+    <pose>0 0 0 0 1.5707 1.5707</pose>
+    <inertial>
+       <mass value="5.0"/>
+          <origin xyz="0 0 0" rpy="0 1.5707 1.5707"/>
+	     <inertia
+		  ixx="0.1" ixy="0" ixz="0"
+		  iyy="0.1" iyz="0"
+		  izz="0.1"
+	      />
+    </inertial>
+    <collision>
+       <origin xyz="0 0 0" rpy="0 1.5707 1.5707" />
+       <geometry>
+          <cylinder radius="0.1" length="0.05" />
+       </geometry>
+    </collision>
+    <visual>
+       <origin xyz="0 0 0" rpy="0 1.5707 1.5707" />
+       <geometry>
+          <cylinder radius="0.1" length="0.05" />
+       </geometry>
+       <material name="green"/>
+    </visual>
+  </link>
+  <!-- Right Wheel Robot chassis joint -->
+  <joint type="continuous" name="right_wheel_hinge">
+    <origin xyz="0 -0.15 0" rpy="0 0 0"/>
+    <child link="right_wheel"/>
+    <parent link="chassis"/>
+    <axis xyz="0 1 0" rpy="0 0 0"/>
+    <limit effort="10000" velocity="1000"/>
+    <joint_properties damping="1.0" friction="1.0"/>
+  </joint>
+  <!-- camera sensor -->
+  <link name="camera">
+    <pose>0 0 0 0 0 0</pose>
+    <inertial>
+       <mass value="0.1"/>
+       <origin xyz="0 0 0" rpy="0 0 0"/>
+       <inertia ixx="1e-6" ixy="0" ixz="0" iyy="1e-6" iyz="0" izz="1e-6" />
+    </inertial>
+    <collision>
+       <origin xyz="0 0 0" rpy="0 0 0"/>
+       <geometry>
+          <box size="0.05 0.05 0.05" />
+       </geometry>
+    </collision>
+    <visual>
+       <origin xyz="0 0 0" rpy="0 0 0"/>
+       <geometry>
+          <box size="0.05 0.05 0.05" />
+       </geometry>
+       <material name="red"/>
+    </visual>
+  </link>
+  <joint type="fixed" name="camera_joint">
+    <origin xyz="0.2 0 0" rpy="0 0 0"/>
+    <child link="camera"/>
+    <parent link="chassis"/>
+    <axis xyz="0 1 0" rpy="0 0 0"/>
+    <limit effort="10000" velocity="1000"/>
+    <joint_properties damping="1.0" friction="1.0"/>
+  </joint>
+  <!-- LIDAR sensor -->
+  <link name="hokuyo">
+    <pose>0 0 0 0 0 0</pose>
+    <inertial>
+       <mass value="0.1"/>
+       <origin xyz="0 0 0" rpy="0 0 0"/>
+       <inertia ixx="1e-6" ixy="0" ixz="0" iyy="1e-6" iyz="0" izz="1e-6" />
+    </inertial>
+    <collision>
+       <origin xyz="0 0 0" rpy="0 0 0"/>
+       <geometry>
+          <box size="0.1 0.1 0.1" />
+       </geometry>
+    </collision>
+    <visual>
+       <origin xyz="0 0 0" rpy="0 0 0"/>
+       <geometry>
+          <mesh filename="package://udacity_bot/meshes/hokuyo.dae"/>
+       </geometry>
+    </visual>
+  </link>
+  <joint type="fixed" name="hokuyo_joint">
+    <origin xyz="0.15 0 0.1" rpy="0 0 0"/>
+    <child link="hokuyo"/>
+    <parent link="chassis"/>
+    <axis xyz="0 1 0" rpy="0 0 0"/>
+    <limit effort="10000" velocity="1000"/>
+    <joint_properties damping="1.0" friction="1.0"/>
+  </joint>
 </robot>
